File: DC-DC converter.kicad_sch (KiCad schematic)
At the start: 19 parts, among them J1 Screw_Terminal_01x02, J2 Screw_Terminal_01x02, U1 LMR33630BDDA

Commit message: Added Images
Parts:
- F1: footprint Fuse:Fuse_Littelfuse_372_D8.50mm -> Fuse:Fuse_1206_3216Metric
Changed lines of the file:
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@@
 			)
 		)
-		(property "Footprint" "Fuse:Fuse_Littelfuse_372_D8.50mm"
+		(property "Footprint" "Fuse:Fuse_1206_3216Metric"
 			(at 76.2 90.678 90)
 			(effects
